File: half_bridge_driver.sch (KiCad schematic (older format))
At the start: 7 parts, among them J1 Conn_01x01_Male, J2 Conn_01x01_Male, U1 ZXGD3003E6, U2 ZXGD3003E6

Commit message: Fixed high driver orientation and added one pad for external wiring.
Connections:
- wire segments 33 -> 35
Changed lines of the file:
@@
 EESchema Schematic File Version 4
+LIBS:half_bridge_driver-cache
 EELAYER 26 0
 EELAYER END
@@
 F 3 "http://www.diodes.com/_files/datasheets/ZXGD3003E6.pdf" H 3300 3400 50  0001 C CNN
 	1    3650 3150
-	-1   0    0    1
+	-1   0    0    -1
 $EndComp
 $Comp
@@
 	8550 3050 8550 3250
 Wire Wire Line
-	3150 3050 3150 3250
-Wire Wire Line
-	3650 2850 5450 2850
-Wire Wire Line
-	3650 3450 5450 3450
-Connection ~ 5450 3450
-Wire Wire Line
 	4150 3250 4250 3250
 Wire Wire Line
@@
 Connection ~ 7550 3250
 Wire Wire Line
-	3150 3250 2900 3250
-Connection ~ 3150 3250
+	3150 3250 3050 3250
 Connection ~ 8550 3250
 Text Label 8900 3250 0    50   ~ 0
@@
 Wire Wire Line
 	6400 2850 7250 2850
+Wire Wire Line
+	3150 3050 3050 3050
+Wire Wire Line
+	3050 3050 3050 3250
+Connection ~ 3050 3250
+Wire Wire Line
+	3050 3250 2900 3250
+Wire Wire Line
+	3650 2850 5450 2850
+Wire Wire Line
+	3650 3450 5450 3450
+Connection ~ 5450 3450
 $EndSCHEMATC

Commit message: Added extra pad to test external wiring.
Connections:
- wire segments 35 -> 33
Changed lines of the file:
@@
 L Device:D D1
 U 1 1 5B5B1EBD
-P 6000 3150
-F 0 "D1" V 6046 3071 50  0000 R CNN
-F 1 "GB01SLT12-214" V 5600 3400 50  0000 R CNN
-F 2 "Diodes_SMD:D_SMB" H 6000 3150 50  0001 C CNN
-F 3 "~" H 6000 3150 50  0001 C CNN
-	1    6000 3150
-	0    -1   -1   0
+P 5950 2850
+F 0 "D1" V 5996 2771 50  0000 R CNN
+F 1 "GB01SLT12-214" V 5550 3100 50  0000 R CNN
+F 2 "Diodes_SMD:D_SMB" H 5950 2850 50  0001 C CNN
+F 3 "~" H 5950 2850 50  0001 C CNN
+	1    5950 2850
+	1    0    0    -1
 $EndComp
 Wire Wire Line
@@
 Wire Wire Line
 	5450 3000 5450 2850
-Wire Wire Line
-	6000 3300 6000 3450
-Wire Wire Line
-	6000 3450 5450 3450
-Wire Wire Line
-	6000 3000 6000 2850
 Wire Wire Line
 	7550 3050 7550 3250
@@
 	7450 3250 7300 3250
 Wire Wire Line
-	6000 2850 6400 2850
-Wire Wire Line
 	6400 3450 6400 3300
 Wire Wire Line
@@
 Wire Wire Line
 	6400 3000 6400 2850
-Connection ~ 6400 2850
 Wire Wire Line
 	6400 2850 7250 2850
@@
 Wire Wire Line
 	3650 3450 5450 3450
-Connection ~ 5450 3450
+Wire Wire Line
+	6100 2850 6400 2850
+Connection ~ 6400 2850
+Wire Wire Line
+	5800 2850 5450 2850
+Connection ~ 5450 2850
 $EndSCHEMATC

Commit message: Added extra pad for input and output driver signals to ease wire soldering.
Parts:
- added J3, J4: Conn_01x01_Male, Wire_Pads:SolderWirePad_single_SMD_5x10mm, symbol Connector:Conn_01x01_Male
Connections:
- wire segments 33 -> 35
Changed lines of the file:
@@
 	5800 2850 5450 2850
 Connection ~ 5450 2850
+$Comp
+L Connector:Conn_01x01_Male J4
+U 1 1 5B647B4C
+P 9100 3050
+F 0 "J4" H 9073 2980 50  0000 R CNN
+F 1 "Conn_01x01_Male" H 9073 3071 50  0000 R CNN
+F 2 "Wire_Pads:SolderWirePad_single_SMD_5x10mm" H 9100 3050 50  0001 C CNN
+F 3 "~" H 9100 3050 50  0001 C CNN
+	1    9100 3050
+	-1   0    0    1
+$EndComp
+Wire Wire Line
+	8900 3050 8900 3250
+$Comp
+L Connector:Conn_01x01_Male J3
+U 1 1 5B648241
+P 2700 3050
+F 0 "J3" H 2673 2980 50  0000 R CNN
+F 1 "Conn_01x01_Male" H 2673 3071 50  0000 R CNN
+F 2 "Wire_Pads:SolderWirePad_single_SMD_5x10mm" H 2700 3050 50  0001 C CNN
+F 3 "~" H 2700 3050 50  0001 C CNN
+	1    2700 3050
+	1    0    0    -1
+$EndComp
+Wire Wire Line
+	2900 3050 2900 3250
 $EndSCHEMATC

Commit message: Added docs.
Other:
- note added: "High-Side MOSFET Driver"
- note added: "Low-Side MOSFET Driver"
- note added: "Power flags"
- moved on the sheet: U1, U2
